Commit message: Update of xacro file

File: pioneer3at-kinect/description/urdf/pioneer3at-kinect.xacro (robot description, xacro)
@@ -10,12 +10,12 @@
 	<link name="base_link">
 		<inertial>
-			<mass value="10.0"/>
-			<origin xyz="0.01 0.01 0.177"/>
-			<inertia ixx="0.3338" ixy="0.0" ixz="0.0"
-				 iyy="0.4783" iyz="0.0"
-				 izz="0.3338"/>
+			<mass value="21.5"/> <!-- P3AT 18.6kg plus three batteries @ 2.4kg each  minus four wheels @ 1.4 kg ea and top plate @ 0.1 kg-->
+			<origin xyz="-0.1 0 0.177"/>
+			<inertia ixx="0.3338" ixy="0.0"     ixz="0.0"
+				              iyy="0.4783"  iyz="0.0"
+				                            izz="0.3338"/>
 		</inertial>
-		<visual name="base_visual">
-			<origin xyz="0.01 0.01 0.177" rpy="0.01 0.01 0.01"/>
+		<visual>
+			<origin xyz="0 0 0.177" rpy="0 0 0"/>
 			<geometry name="pioneer_geom">
 				<mesh filename="package://pioneer_kinect_description/meshes/p3at_meshes/chassis.stl"/>
@@ -26,5 +26,5 @@
 		</visual>
 		<collision>
-			<origin xyz="0.01 0.01 0.177" rpy="0.01 0.01 0.01"/>
+			<origin xyz="0 0 0.177" rpy="0 0 0"/>
 				<geometry>
 					<mesh filename="package://pioneer_kinect_description/meshes/p3at_meshes/chassis.stl"/>
@@ -44,6 +44,6 @@
  				izz="1.0"/>
 		</inertial>
-		<visual name="base_visual">
-			<origin xyz="0.01 0.01 0.01" rpy="0.01 0.01 0.01"/>
+		<visual>
+			<origin xyz="0 0 0" rpy="0 0 0"/>
 			<geometry name="pioneer_geom">
 				<mesh filename="package://pioneer_kinect_description/meshes/p3at_meshes/top.stl"/>
@@ -53,10 +53,4 @@
 			</material>
 		</visual>
-		<collision>
-			<origin xyz="0.01 0.01 0.01" rpy="0.01 0.01 0.01"/>
-			<geometry>
-				<box size="0.01 0.01 0.01"/>
-			</geometry>
-		</collision>
 	</link>
 	<gazebo reference="top_plate">
@@ -64,5 +58,5 @@
 	</gazebo>
 	<joint name="base_top_joint" type="fixed">
-		<origin xyz="0.003 0 0.274" rpy="0.01 0.01 0.01"/>
+		<origin xyz="0.003 0 0.274" rpy="0 0 0"/>
 		<parent link="base_link"/>
 		<child link="top_plate"/>
@@ -72,10 +66,10 @@
 		<inertial>
 			<mass value="0.1"/>
-			<origin xyz="0.01 0.01 0.01"/>
+			<origin xyz="0 0 0"/>
 			<inertia ixx="1.0" ixy="0.0" ixz="0.0"
 				 iyy="1.0" iyz="0.0" izz="1.0"/>
 		</inertial>
 		<visual name="base_visual">
-			<origin xyz="0.01 0.01 0.01" rpy="0.01 0.01 0.01"/>
+			<origin xyz="0 0 0" rpy="0 0 0"/>
 			<geometry name="pioneer_geom">
 				<mesh filename="package://pioneer_kinect_description/meshes/p3at_meshes/front_sonar.stl"/>
@@ -85,10 +79,4 @@
 			</material>
 		</visual>
-		<collision>
-			<origin xyz="0.01 0.01 0.01" rpy="0.01 0.01 0.01"/>
-			<geometry>
-				<box size="0.01 0.01 0.01"/>
-			</geometry>
-		</collision>
 	</link>
 	<gazebo reference="front_sonar">
@@ -96,5 +84,5 @@
 	</gazebo>
 	<joint name="base_front_joint" type="fixed">
-		<origin xyz="0.193 0 0.25" rpy="0.01 0.01 0.01"/>
+		<origin xyz="0.193 0 0.25" rpy="0 0 0"/>
 		<parent link="base_link"/>
 		<child link="front_sonar"/>
@@ -103,10 +91,10 @@
 		<inertial>
 			<mass value="0.1"/>
-			<origin xyz="0.01 0.01 0.01"/>
+			<origin xyz="0 0 0"/>
 			<inertia ixx="1.0" ixy="0.0" ixz="0.0"
 				 iyy="1.0" iyz="0.0" izz="1.0"/>
 		</inertial>
 		<visual name="base_visual">
-			<origin xyz="0.01 0.01 0.01" rpy="0.01 0.01 0.01"/>
+			<origin xyz="0 0 0" rpy="0 0 0"/>
 			<geometry name="pioneer_geom">
 				<mesh filename="package://pioneer_kinect_description/meshes/p3at_meshes/back_sonar.stl"/>
@@ -116,10 +104,4 @@
 			</material>
 		</visual>
-		<collision>
-			<origin xyz="0.01 0.01 0.01" rpy="0.01 0.01 0.01"/>
-			<geometry>
-				<box size="0.01 0.01 0.01"/>
-			</geometry>
-		</collision>
 	</link>
 	<gazebo reference="back_sonar">
@@ -127,5 +109,5 @@
 	</gazebo>
 	<joint name="base_back_joint" type="fixed">
-		<origin xyz="-0.187 0 0.247" rpy="0.01 0.01 0.01"/>
+		<origin xyz="-0.187 0 0.247" rpy="0 0 0"/>
 		<parent link="base_link"/>
 		<child link="back_sonar"/>
@@ -136,10 +118,10 @@
 		<inertial>
 			<mass value="0.1"/>
-			<origin xyz="0.01 0.01 0.01"/>
+			<origin xyz="0 0 0"/>
 			<inertia ixx="1.0" ixy="0.0" ixz="0.0"
 				 iyy="1.0" iyz="0.0" izz="1.0"/>
   	 	</inertial>
-		<visual name="base_visual">
-			<origin xyz="0.01 0.01 0.01" rpy="0.01 0.01 0.01"/>
+		<visual>
+			<origin xyz="0 0 0" rpy="0 0 0"/>
 			<geometry name="pioneer_geom">
 				<mesh filename="package://pioneer_kinect_description/meshes/p3at_meshes/axle.stl"/>
@@ -149,10 +131,4 @@
 			</material>
 		</visual>
-		<collision>
-			<origin xyz="0.01 0.01 0.01" rpy="0.01 0.01 0.01"/>
-			<geometry>
-				<box size="0.01 0.01 0.01"/>
-			</geometry>
-		</collision>
 	</link>
 	<gazebo reference="p3at_front_${suffix}_axle">
@@ -160,5 +136,5 @@
 	</gazebo>
 	<joint name="base_front_${suffix}_axle_joint" type="fixed">
-		<origin xyz="0.135 ${reflect*0.156} 0.111" rpy="0.01 0.01 0.01"/>
+		<origin xyz="0.135 ${reflect*0.156} 0.111" rpy="0 0 0"/>
 		<parent link="base_link"/>
 		<child link="p3at_front_${suffix}_axle"/>
@@ -167,10 +143,10 @@
 		<inertial>
 			<mass value="0.1"/>
-			<origin xyz="0.01 0.01 0.01"/>
+			<origin xyz="0 0 0"/>
 			<inertia ixx="1.0" ixy="0.0" ixz="0.0"
 				 iyy="1.0" iyz="0.0" izz="1.0"/>
   	 	</inertial>
-		<visual name="base_visual">
-			<origin xyz="0.01 0.01 0.01" rpy="0.01 0.01 0.01"/>
+		<visual>
+			<origin xyz="0 0 0" rpy="0 0 0"/>
 			<geometry name="pioneer_geom">
 				<mesh filename="package://pioneer_kinect_description/meshes/p3at_meshes/${suffix}_hubcap.stl"/>
@@ -180,10 +156,4 @@
 			</material>
 		</visual>
-		<collision>
-			<origin xyz="0.01 0.01 0.01" rpy="0.01 0.01 0.01"/>
-			<geometry>
-				<box size="0.01 0.01 0.01"/>
-			</geometry>
-		</collision>
 	</link>
 	<gazebo reference="p3at_front_${suffix}_hub">
@@ -191,5 +161,5 @@
 	</gazebo>
 	<joint name="base_front_${suffix}_hub_joint" type="fixed">
-		<origin xyz="0 ${reflect*0.041} 0" rpy="0.01 0.01 0.01"/>
+		<origin xyz="0 ${reflect*0.041} 0" rpy="0 0 0"/>
 		<parent link="p3at_front_${suffix}_axle"/>
 		<child link="p3at_front_${suffix}_hub"/>
@@ -197,11 +167,11 @@
 	<link name="p3at_front_${suffix}_wheel">
 		<inertial>
-			<mass value="0.5"/>
-			<origin xyz="0.01 0.01 0.01"/>
+			<mass value="1.2"/> <!-- 1.4 kg - axle 0.1 kg - hub 0.1 kg -->
+			<origin xyz="0 0 0"/>
 			<inertia ixx="0.012411765597" ixy="0" ixz="0"
          iyy="0.015218160428" iyz="0" izz="0.011763977943"/>
-      </inertial>
-		<visual name="base_visual">
-			<origin xyz="0.01 0.01 0.01" rpy="0.01 0.01 0.01"/>
+      	</inertial>
+		<visual>
+			<origin xyz="0 0 0" rpy="0 0 0"/>
 			<geometry name="pioneer_geom">
 				<mesh filename="package://pioneer_kinect_description/meshes/p3at_meshes/wheel.stl"/>
@@ -212,7 +182,8 @@
 		</visual>
 		<collision>
-			<origin xyz="0.01 0.01 0.01" rpy="${-(pi/2)} 0 0"/>
+			<origin xyz="0 0 0" rpy="${-3.1415927/2} 0 0"/>
 			<geometry>
-	    	    <cylinder radius="0.111" length="0.075"/>
+		    <!--mesh filename="package://amr_robots_description/meshes/p3at_meshes/wheel.stl"/-->
+		    <cylinder radius="0.111" length="0.075"/>
 			</geometry>
 		</collision>
@@ -223,6 +194,6 @@
 	<joint name="p3at_front_${suffix}_wheel_joint" type="continuous">
  		<axis xyz="0 1 0"/>
-       	<anchor xyz="0.01 0.01 0.01"/>
-		<origin xyz="0.01 0.01 0.01" rpy="0.01 0.01 0.01"/>
+       	<anchor xyz="0 0 0"/>
+		<origin xyz="0 0 0" rpy="0 0 0"/>
 		<parent link="p3at_front_${suffix}_hub"/>
 		<child link="p3at_front_${suffix}_wheel"/>
@@ -234,10 +205,10 @@
 		<inertial>
 			<mass value="0.1"/>
-			<origin xyz="0.01 0.01 0.01"/>
+			<origin xyz="0 0 0"/>
 			<inertia ixx="1.0" ixy="0.0" ixz="0.0"
 				 iyy="1.0" iyz="0.0" izz="1.0"/>
   	 	</inertial>
-		<visual name="base_visual">
-			<origin xyz="0.01 0.01 0.01" rpy="0.01 0.01 0.01"/>
+		<visual>
+			<origin xyz="0 0 0" rpy="0 0 0"/>
 			<geometry name="pioneer_geom">
 				<mesh filename="package://pioneer_kinect_description/meshes/p3at_meshes/axle.stl"/>
@@ -248,5 +219,5 @@
 		</visual>
 		<collision>
-			<origin xyz="0.01 0.01 0.01" rpy="0.01 0.01 0.01"/>
+			<origin xyz="0 0 0" rpy="0 0 0"/>
 			<geometry>
 				<mesh filename="package://pioneer_kinect_description/meshes/p3at_meshes/axle.stl"/>
@@ -258,5 +229,5 @@
 	</gazebo>
 	<joint name="p3at_back_${suffix}_axle_joint" type="fixed">
-		<origin xyz="-0.134 ${reflect*0.156} 0.111" rpy="0.01 0.01 0.01"/>
+		<origin xyz="-0.134 ${reflect*0.156} 0.111" rpy="0 0 0"/>
 		<parent link="base_link"/>
 		<child link="p3at_back_${suffix}_axle"/>
@@ -265,10 +236,10 @@
 		<inertial>
 			<mass value="0.1"/>
-			<origin xyz="0.01 0.01 0.01"/>
+			<origin xyz="0 0 0"/>
 			<inertia ixx="1.0" ixy="0.0" ixz="0.0"
 				 iyy="1.0" iyz="0.0" izz="1.0"/>
   	 	</inertial>
-		<visual name="base_visual">
-			<origin xyz="0.01 0.01 0.01" rpy="0.01 0.01 0.01"/>
+		<visual>
+			<origin xyz="0 0 0" rpy="0 0 0"/>
 			<geometry name="pioneer_geom">
 				<mesh filename="package://pioneer_kinect_description/meshes/p3at_meshes/${suffix}_hubcap.stl"/>
@@ -277,5 +248,5 @@
 		</visual>
 		<collision>
-			<origin xyz="0.01 0.01 0.01" rpy="0.01 0.01 0.01"/>
+			<origin xyz="0 0 0" rpy="0 0 0"/>
 			<geometry>
 				<mesh filename="package://pioneer_kinect_description/meshes/p3at_meshes/${suffix}_hubcap.stl"/>
@@ -287,5 +258,5 @@
 	</gazebo>
  	<joint name="p3at_back_${suffix}_hub_joint" type="fixed">
-		<origin xyz="-0 ${reflect*0.041} 0" rpy="0.01 0.01 0.01"/>
+		<origin xyz="-0 ${reflect*0.041} 0" rpy="0 0 0"/>
 		<parent link="p3at_back_${suffix}_axle"/>
 		<child link="p3at_back_${suffix}_hub"/>
@@ -293,11 +264,11 @@
 	<link name="p3at_back_${suffix}_wheel">
 		<inertial>
-			<mass value="0.5"/>
-			<origin xyz="0.01 0.01 0.01"/>
+			<mass value="1.2"/>
+			<origin xyz="0 0 0"/>
 			<inertia ixx="0.012411765597" ixy="0" ixz="0"
         	 iyy="0.015218160428" iyz="0" izz="0.011763977943"/>
     	</inertial>
-		<visual name="base_visual">
-			<origin xyz="0.01 0.01 0.01" rpy="0.01 0.01 0.01"/>
+		<visual>
+			<origin xyz="0 0 0" rpy="0 0 0"/>
 			<geometry name="pioneer_geom">
 				<mesh filename="package://pioneer_kinect_description/meshes/p3at_meshes/wheel.stl"/>
@@ -306,5 +277,5 @@
 		</visual>
 		<collision>
-			<origin xyz="0.01 0.01 0.01" rpy="${-(pi/2)} 0 0"/>
+			<origin xyz="0 0 0" rpy="${-(pi/2)} 0 0"/>
 			<geometry>
 	        	<cylinder radius="0.111" length="0.075"/>
@@ -317,42 +288,46 @@
 	<joint name="p3at_back_${suffix}_wheel_joint" type="continuous">
 		<axis xyz="0 1 0"/>
-        <anchor xyz="0.01 0.01 0.01"/>
+        <anchor xyz="0 0 0"/>
         <limit effort="100" velocity="100" />
         <joint_properties damping="0.7"/>
-		<origin xyz="0.01 0.01 0.01" rpy="0.01 0.01 0.01"/>
+		<origin xyz="0 0 0" rpy="0 0 0"/>
 		<parent link="p3at_back_${suffix}_hub"/>
 		<child link="p3at_back_${suffix}_wheel"/>
 	</joint>
-	<gazebo reference="p3at_back_${suffix}_wheel">
-    	<kp>1000000.0</kp> <!-- kp and kd for rubber -->
-    	<kd>100.0</kd>
-    	<mu1>10.0</mu1>
-    	<mu2>1.0</mu2>
-    	<fdir1>0 1 0</fdir1> <!-- is this correct? -->
-    	<maxVel>1.0</maxVel>
-    	<minDepth>0.00</minDepth>
-  	</gazebo>
- 	<gazebo reference="p3at_front_${suffix}_wheel">
-    	<kp>1000000.0</kp> <!-- kp and kd for rubber -->
-    	<kd>100.0</kd>
-    	<mu1>10.0</mu1>
-    	<mu2>1.0</mu2>
-    	<fdir1>0 1 0</fdir1> <!-- is this correct? -->
-    	<maxVel>1.0</maxVel>
-    	<minDepth>0.00</minDepth>
-  	</gazebo>
+  	  <!-- see http://gazebosim.org/tutorials/?tut=ros_urdf -->
+  <gazebo reference="p3at_back_${suffix}_wheel">
+    <kp>1000000.0</kp> <!-- kp and kd for rubber -->
+    <kd>100.0</kd>
+    <mu1>1.0</mu1> <!-- was 10 -->
+    <mu2>1.0</mu2>
+      <!-- how to get these into <surface><friction><ode>... ?
+        slip1 0.5 /slip1
+         slip2 0 /slip2
+      -->
+    <!-- fdir1 0 1 0 /fdir1 --> <!-- see http://github.com/MobileRobots/amr-ros-config/issues/6 -->
+    <maxVel>1.0</maxVel>
+    <minDepth>0.00</minDepth>
+    <material value="Gazebo/Black" />
+  </gazebo>
+  <gazebo reference="p3at_front_${suffix}_wheel">
+    <kp>1000000.0</kp> <!-- kp and kd for rubber -->
+    <kd>100.0</kd>
+    <mu1>1.0</mu1> <!-- was 10 -->
+    <mu2>1.0</mu2>
+      <!-- how to get these into <surface><friction><ode>... ?
+        slip1 0.5 /slip1
+         slip2 0 /slip2
+      -->
+    <!-- fdir1 0 1 0 /fdir1 --> <!-- see http://github.com/MobileRobots/amr-ros-config/issues/6 -->
+    <maxVel>1.0</maxVel>
+    <minDepth>0.00</minDepth>
+    <material value="Gazebo/Black" />
+  </gazebo>
 </xacro:macro>
 <xacro:macro name="p3at_gazebo_ext">
-	<gazebo>
-    	<plugin name="joint_state_publisher" filename="libgazebo_ros_joint_state_publisher.so">
-        	<robotNamespace></robotNamespace>
-        	<jointName>p3at_front_left_wheel_joint, p3at_front_right_wheel_joint, p3at_back_left_wheel_joint, p3at_back_right_wheel_joint</jointName>
-        	<updateRate>10.0</updateRate>
-        	<alwaysOn>true</alwaysOn>
-      	</plugin>
-  	</gazebo>
+  	<!--Gazebo Differential Drive Plugin-->
 	<gazebo>
   		<plugin name="skid_steer_drive_controller" filename="libgazebo_ros_skid_steer_drive.so">
-    		<updateRate>0.0</updateRate>
+    		<updateRate>20.0</updateRate>
     		<robotNamespace>/</robotNamespace>
     		<leftFrontJoint>p3at_front_left_wheel_joint</leftFrontJoint>
@@ -363,7 +338,10 @@
     		<wheelDiameter>0.215</wheelDiameter>
     		<robotBaseFrame>base_link</robotBaseFrame>
-    		<torque>20</torque>
+    		<torque>200</torque>
     		<topicName>cmd_vel</topicName>
     		<odometryFrame>odom</odometryFrame>
+    		<covariance_x>0.0001</covariance_x>
+    		<covariance_y>0.0001</covariance_y>
+    		<covariance_yaw>0.01</covariance_yaw>
     		<broadcastTF>true</broadcastTF>
   		</plugin>
